File: board/belt.sch (KiCad schematic (older format))
At the start: 25 parts, among them J1 USB_B_Micro, J2 USB_B_Micro, J3 USB_B_Micro, J4 USB_B_Micro, P1 3352T-1-103LF, P2 3352T-1-103LF, Q1 BSS138, Q2 BSS138, SW1 SW_SPDT, SW2 SW_Push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

Commit message: fix schematic symbol which was using old POT symbol
Parts:
- P1, P2: value 3352T-1-103LF -> 10K; symbol belt-rescue:3352T-1-103LF-3352T-1-103LF -> Device:R_POT
Changed lines of the file:
@@
 BUTTON
-$Comp
-L belt-rescue:3352T-1-103LF-3352T-1-103LF P1
-U 1 1 5E3B3B17
-P 1500 1050
-F 0 "P1" H 1500 1165 50  0000 C CNN
-F 1 "3352T-1-103LF" H 1500 1256 50  0000 C CNN
-F 2 "Potentiometer_THT:PDB12-H" H 1500 1050 50  0001 L BNN
-F 3 "" H 1500 1050 50  0001 L BNN
-F 4 "IPC-7351B" H 1500 1050 50  0001 L BNN "Field4"
-F 5 "08/19" H 1500 1050 50  0001 L BNN "Field5"
-F 6 "Bourns" H 1500 1050 50  0001 L BNN "Field6"
-	1    1500 1050
-	-1   0    0    1
-$EndComp
 $Comp
 L power:GND #PWR0122
 U 1 1 5E3B56F0
-P 1200 1050
-F 0 "#PWR0122" H 1200 800 50  0001 C CNN
-F 1 "GND" V 1205 922 50  0000 R CNN
-F 2 "" H 1200 1050 50  0001 C CNN
-F 3 "" H 1200 1050 50  0001 C CNN
-	1    1200 1050
-	0    1    1    0
+P 1650 1050
+F 0 "#PWR0122" H 1650 800 50  0001 C CNN
+F 1 "GND" V 1655 922 50  0000 R CNN
+F 2 "" H 1650 1050 50  0001 C CNN
+F 3 "" H 1650 1050 50  0001 C CNN
+	1    1650 1050
+	0    -1   -1   0
 $EndComp
 Text Label 6150 3150 3    50   ~ 0
 THUMBDIAL2
-Text Label 1500 850  0    50   ~ 0
+Text Label 1500 900  0    50   ~ 0
 THUMBDIAL1
 $Comp
@@
 NoConn ~ 1700 2650
 $Comp
-L belt-rescue:3352T-1-103LF-3352T-1-103LF P2
+L Device:R_POT P2
 U 1 1 5E3E27DC
 P 1500 1600
-F 0 "P2" H 1500 1715 50  0000 C CNN
-F 1 "3352T-1-103LF" H 1500 1806 50  0000 C CNN
+F 0 "P2" V 1300 1600 50  0000 C CNN
+F 1 "10K" V 1400 1600 50  0000 C CNN
 F 2 "Potentiometer_THT:PDB12-H" H 1500 1600 50  0001 L BNN
 F 3 "" H 1500 1600 50  0001 L BNN
@@
 F 6 "Bourns" H 1500 1600 50  0001 L BNN "Field6"
 	1    1500 1600
-	-1   0    0    1
+	0    -1   -1   0
 $EndComp
 $Comp
 L power:GND #PWR0133
 U 1 1 5E3E27E2
-P 1200 1600
-F 0 "#PWR0133" H 1200 1350 50  0001 C CNN
-F 1 "GND" V 1205 1472 50  0000 R CNN
-F 2 "" H 1200 1600 50  0001 C CNN
-F 3 "" H 1200 1600 50  0001 C CNN
-	1    1200 1600
-	0    1    1    0
-$EndComp
-Text Label 1500 1400 0    50   ~ 0
+P 1650 1600
+F 0 "#PWR0133" H 1650 1350 50  0001 C CNN
+F 1 "GND" V 1655 1472 50  0000 R CNN
+F 2 "" H 1650 1600 50  0001 C CNN
+F 3 "" H 1650 1600 50  0001 C CNN
+	1    1650 1600
+	0    -1   -1   0
+$EndComp
+Text Label 1500 1450 0    50   ~ 0
 THUMBDIAL2
 Text Label 6650 950  1    50   ~ 0
@@
 L power:+3.3VA #PWR0110
 U 1 1 5E3FC6B5
-P 1800 1050
-F 0 "#PWR0110" H 1800 900 50  0001 C CNN
-F 1 "+3.3VA" V 1815 1178 50  0000 L CNN
-F 2 "" H 1800 1050 50  0001 C CNN
-F 3 "" H 1800 1050 50  0001 C CNN
-	1    1800 1050
-	0    1    1    0
+P 1350 1050
+F 0 "#PWR0110" H 1350 900 50  0001 C CNN
+F 1 "+3.3VA" V 1350 1150 50  0000 L CNN
+F 2 "" H 1350 1050 50  0001 C CNN
+F 3 "" H 1350 1050 50  0001 C CNN
+	1    1350 1050
+	0    -1   -1   0
 $EndComp
 $Comp
 L power:+3.3VA #PWR0114
 U 1 1 5E401221
-P 1800 1600
-F 0 "#PWR0114" H 1800 1450 50  0001 C CNN
-F 1 "+3.3VA" V 1815 1728 50  0000 L CNN
-F 2 "" H 1800 1600 50  0001 C CNN
-F 3 "" H 1800 1600 50  0001 C CNN
-	1    1800 1600
-	0    1    1    0
+P 1350 1600
+F 0 "#PWR0114" H 1350 1450 50  0001 C CNN
+F 1 "+3.3VA" V 1350 1700 50  0000 L CNN
+F 2 "" H 1350 1600 50  0001 C CNN
+F 3 "" H 1350 1600 50  0001 C CNN
+	1    1350 1600
+	0    -1   -1   0
 $EndComp
 $Comp
@@
 	1    0    0    -1
 $EndComp
+$Comp
+L Device:R_POT P1
+U 1 1 5E3B3B17
+P 1500 1050
+F 0 "P1" V 1300 1050 50  0000 C CNN
+F 1 "10K" V 1400 1050 50  0000 C CNN
+F 2 "Potentiometer_THT:PDB12-H" H 1500 1050 50  0001 L BNN
+F 3 "" H 1500 1050 50  0001 L BNN
+F 4 "IPC-7351B" H 1500 1050 50  0001 L BNN "Field4"
+F 5 "08/19" H 1500 1050 50  0001 L BNN "Field5"
+F 6 "Bourns" H 1500 1050 50  0001 L BNN "Field6"
+	1    1500 1050
+	0    -1   -1   0
+$EndComp
 $EndSCHEMATC

Commit message: scoot pots apart to sorta be able to fit plastic tops
Parts:
- SW2: footprint Button_Switch_SMD:SW_Push_1P1T_NO_6x6mm_H9.5mm -> Button_Switch_THT:SW_PUSH_6mm_H5mm
Changed lines of the file:
@@
 F 0 "SW2" H 1500 2585 50  0000 C CNN
 F 1 "SW_Push" H 1500 2494 50  0000 C CNN
-F 2 "Button_Switch_SMD:SW_Push_1P1T_NO_6x6mm_H9.5mm" H 1500 2500 50  0001 C CNN
+F 2 "Button_Switch_THT:SW_PUSH_6mm_H5mm" H 1500 2500 50  0001 C CNN
 F 3 "~" H 1500 2500 50  0001 C CNN
 	1    1500 2300

Commit message: move several belt footprints into local belt footprint library; fix footprints for power switch and BNO055 which had through-holes that were too small
Parts:
- P1, P2: footprint Potentiometer_THT:PDB12-H -> belt:PDB12-H
- SW1: footprint Extra SMD Components:Button_Switch_SPDT_GH36P010001 -> belt:Button_Switch_SPDT_GH36P010001
Changed lines of the file:
@@
 EESchema Schematic File Version 4
-LIBS:belt-cache
-EELAYER 29 0
+EELAYER 30 0
 EELAYER END
 $Descr A4 11693 8268
@@
 F 0 "P2" V 1300 1600 50  0000 C CNN
 F 1 "10K" V 1400 1600 50  0000 C CNN
-F 2 "Potentiometer_THT:PDB12-H" H 1500 1600 50  0001 L BNN
+F 2 "belt:PDB12-H" H 1500 1600 50  0001 L BNN
 F 3 "" H 1500 1600 50  0001 L BNN
 F 4 "IPC-7351B" H 1500 1600 50  0001 L BNN "Field4"
@@
 F 0 "SW1" H 1500 3035 50  0000 C CNN
 F 1 "SW_SPDT" H 1500 2944 50  0000 C CNN
-F 2 "Extra SMD Components:Button_Switch_SPDT_GH36P010001" H 1500 2750 50  0001 C CNN
+F 2 "belt:Button_Switch_SPDT_GH36P010001" H 1500 2750 50  0001 C CNN
 F 3 "~" H 1500 2750 50  0001 C CNN
 	1    1500 2750
@@
 F 0 "P1" V 1300 1050 50  0000 C CNN
 F 1 "10K" V 1400 1050 50  0000 C CNN
-F 2 "Potentiometer_THT:PDB12-H" H 1500 1050 50  0001 L BNN
+F 2 "belt:PDB12-H" H 1500 1050 50  0001 L BNN
 F 3 "" H 1500 1050 50  0001 L BNN
 F 4 "IPC-7351B" H 1500 1050 50  0001 L BNN "Field4"
